Commit message: newMap

File: description/robot_core.xacro (robot description, xacro)
@@ -3,4 +3,12 @@
     <!-- Example link -->
     <xacro:include filename="inertial_macros.xacro"/>
+    <!-- Example link -->
+    <link name="base_footprint">
+    </link>
+    <joint name="base_footprint_joint" type="fixed">
+        <parent link="base_link"/>
+        <child link="base_footprint"/>
+        <origin xyz="0 0 0"/>
+    </joint>
     <!-- Example link -->
     <link name="base_link">

Commit message: slam

File: description/robot_core.xacro (robot description, xacro)
@@ -3,7 +3,15 @@
     <!-- Example link -->
     <xacro:include filename="inertial_macros.xacro"/>
-    <!-- Example link -->
+   <!-- Example link -->
     <link name="base_link">
     </link>
+    <!-- Example link -->
+    <link name="base_footprint">
+    </link>
+ <joint name="base_footprint_joint" type="fixed">
+        <parent link="base_link"/>
+        <child link="base_footprint"/>
+        <origin xyz="0 0 0"/>
+    </joint>
     <joint name="base_link" type="fixed">
         <parent link="base_link"/>
